File: Tang Primer 20k HD6309 Board.kicad_pcb (KiCad board)
At the start: 2 copper layers, 87.6 x 48.3 mm, 17 parts, among them J1 TANG PRIMER 20K, J2 5V, U1 MC6809, U2 74LVC16245A, U3 74LVC16245A

Commit message: WIP
Parts:
- removed J1: TANG PRIMER 20K, Connector_PinSocket_2.54mm:PinSocket_2x20_P2.54mm_Vertical
- removed J2: 5V, Connector_PinHeader_2.54mm:PinHeader_1x02_P2.54mm_Vertical
- added C10: 100nF, Capacitor_SMD:C_0805_2012Metric, F.Cu at (94.3, 176.6)
- added C11: 220uF, Capacitor_SMD:CP_Elec_6.3x7.7, F.Cu at (75.2, 33.8)
- added C12: 0.1uF, Capacitor_SMD:C_0805_2012Metric, F.Cu at (56.9, 45.5)
- added C8: 100nF, Capacitor_SMD:C_0805_2012Metric, F.Cu at (120.9, 154.3)
- added C9: 100nF, Capacitor_SMD:C_0805_2012Metric, F.Cu at (116.4, 154.3)
- added H1: MountingHole_Pad, MountingHole:MountingHole_3.2mm_M3_Pad_Via, F.Cu at (156.0, 140.8)
- added H2: MountingHole_Pad, MountingHole:MountingHole_3.2mm_M3_Pad_Via, F.Cu at (48.2, 141.0)
- added H3: MountingHole_Pad, MountingHole:MountingHole_3.2mm_M3_Pad_Via, F.Cu at (156.2, 33.4)
- added H4: MountingHole_Pad, MountingHole:MountingHole_3.2mm_M3_Pad_Via, F.Cu at (48.2, 33.2)
- added J3: JTAG, Connector_PinHeader_2.54mm:PinHeader_2x06_P2.54mm_Vertical, F.Cu at (85.4, 34.9)
- added J4: USB-C, Connector_USB:USB_C_Receptacle_HRO_TYPE-C-31-M-12, F.Cu at (61.8, 31.1)
- added PRIMER_20K_1: ~, primer20k:DDR3-SMD_0705F0BE40F, F.Cu at (67.0, 88.2)
- added R3: 10k, Resistor_SMD:R_0805_2012Metric, B.Cu at (60.0, 131.9)
- added R4: 5.11k, Resistor_SMD:R_0805_2012Metric, F.Cu at (59.5, 39.0)
- added R5: 5.11k, Resistor_SMD:R_0805_2012Metric, F.Cu at (63.9, 39.0)
- added R6: 10k, Resistor_SMD:R_0805_2012Metric, B.Cu at (60.0, 128.3)
- added R7: 10k, Resistor_SMD:R_0805_2012Metric, F.Cu at (129.7, 133.1)
- added R8: 50, Resistor_SMD:R_0805_2012Metric, F.Cu at (102.9, 171.6)
- added SW1: FPGA_RST, Button_Switch_SMD:SW_SPST_CK_RS282G05A3, F.Cu at (60.5, 139.2)
- added SW2: MPU_RST, Button_Switch_SMD:SW_SPST_CK_RS282G05A3, F.Cu at (69.0, 139.2)
- added SW3: CONFIG, Button_Switch_SMD:SW_DIP_SPSTx04_Slide_KingTek_DSHP04TS_W7.62mm_P1.27mm, F.Cu at (80.6, 139.1)
- added TP1: EXTAL, TestPoint:TestPoint_Loop_D1.80mm_Drill1.0mm_Beaded, F.Cu at (136.1, 68.9)
- added TP2: Q, TestPoint:TestPoint_Loop_D1.80mm_Drill1.0mm_Beaded, F.Cu at (135.9, 76.2)
- added TP3: E, TestPoint:TestPoint_Loop_D1.80mm_Drill1.0mm_Beaded, F.Cu at (142.3, 80.0)
- added TP4: R/~{W}, TestPoint:TestPoint_Loop_D1.80mm_Drill1.0mm_Beaded, F.Cu at (135.9, 84.5)
- added U4: CH340E, Package_SO:MSOP-10_3x3mm_P0.5mm, F.Cu at (61.0, 45.8)
- C2, C3, C4, C5, C6: moved to F.Cu
- C7: value 1uF -> 10uF; moved to F.Cu
- R1: value 1k -> 150
- RN1: footprint Resistor_SMD:R_Array_Convex_5x1206 -> Resistor_SMD:R_Array_Convex_5x0603
- moved D1 75.9 mm to (57.7, 156.1), turned to -90 degrees
- moved C7 74.2 mm to (105.6, 165.5), turned to 0 degrees
- moved C6 70.2 mm to (95.0, 139.6)
- moved R2 67.7 mm to (105.6, 168.5)
- moved RN1 66.6 mm to (118.0, 69.1)
- moved R1 66.1 mm to (70.4, 158.1)
- moved C5 58.5 mm to (95.3, 68.8), turned to 0 degrees
- moved C4 58.4 mm to (95.3, 84.5), turned to 0 degrees
- moved U1 56.8 mm to (110.4, 63.9), turned to 0 degrees
- moved U3 56.8 mm to (95.5, 76.6)
- moved C1 36.4 mm to (107.5, 78.3), turned to 90 degrees
- moved D2 34.6 mm to (125.3, 133.1), turned to 0 degrees
- moved C2 15.8 mm to (95.3, 106.5), turned to 0 degrees
- moved C3 10.4 mm to (95.3, 90.9), turned to 0 degrees
- moved U2 4.74 mm to (95.3, 98.6), turned to 0 degrees
Connections:
- RN1 pad 2: ~{RESET} -> ~{FIRQ}
- RN1 pad 3: ~{NMI} -> ~{IRQ}
- RN1 pad 4: ~{IRQ} -> unconnected-(RN1-Pad4)
- RN1 pad 5: ~{FIRQ} -> ~{NMI}
- RN1 pad 6: ~{DMA/BREQ} -> ~{HALT}
- RN1 pad 7: ~{HALT} -> ~{RESET}
- RN1 pad 9: unconnected-(RN1-Pad9) -> ~{DMA/BREQ}
- U1 pad 38: EXTAL -> Net-(R8-Pad1)
Routing:
- net +5V: track 102.3 -> 0.00 mm, vias 2 -> 0
- net ~{RESET}: track 75.2 -> 0.00 mm, vias 3 -> 0
- net /BUF_A0: track 74.7 -> 0.00 mm, vias 3 -> 0
- net EXTAL: track 73.2 -> 0.00 mm
- net /BUF_A1: track 71.5 -> 0.00 mm, vias 1 -> 0
- net /BUF_A2: track 69.0 -> 0.00 mm, vias 1 -> 0
- net /BUF_A3: track 67.0 -> 0.00 mm, vias 1 -> 0
- net GND: track 66.4 -> 0.00 mm, vias 22 -> 0
- net /D7: track 60.9 -> 0.00 mm
- net /D6: track 58.2 -> 0.00 mm
- net /BUF_A5: track 56.0 -> 0.00 mm, vias 1 -> 0
- net /D5: track 55.2 -> 0.00 mm
- net /BUF_A4: track 54.4 -> 0.00 mm, vias 1 -> 0
- net /BUF_A6: track 54.0 -> 0.00 mm, vias 1 -> 0
- net /D4: track 52.5 -> 0.00 mm
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- added copper zone on F.Cu, net GND
- removed copper zone on F.Cu, net +3V3
- removed copper zone on B.Cu, net GND
Other:
- board size 87.6 x 48.3 mm -> 120 x 120 mm
- board text added: "6809"
- board text removed: "3V3"
- board text removed: "6809 Sidecar"
- board text removed: "@markbaseggio"
- board text removed: "A0"
- board text removed: "A1"
- board text removed: "A10"
- board text removed: "A11"
- board text removed: "A12"
- board text removed: "A13"
- board text removed: "A14"
- board text removed: "A15"
- board text removed: "A2"
- board text removed: "A3"
- board text removed: "A4"
- board text removed: "A5"
- board text removed: "A6"
- board text removed: "A7"
- board text removed: "A8"
- board text removed: "A9"
- board text removed: "D0"
- board text removed: "D1"
- board text removed: "D2"
- board text removed: "D3"
- board text removed: "D4"
- board text removed: "D5"
- board text removed: "D6"
- board text removed: "D7"
- board text removed: "DIR"
- board text removed: "E"
- board text removed: "EXTAL"
- board text removed: "GND"
- board text removed: "RST"
- board text removed: "RW"
- board text removed: "TCK"
- board text removed: "TDI"
- board text removed: "TDO"
- board text removed: "TMS"
- board text removed: "r1"
