File: Tang Primer 20k HD6309 Board.kicad_pcb (KiCad board)
At the start: 2 copper layers, 120 x 120 mm, 41 parts, among them J3 JTAG, J4 USB-C, SW1 FPGA_RST, SW2 MPU_RST, SW3 CONFIG, U1 MC6809, U2 74LVC16245A, U3 74LVC16245A, U4 CH340E

Commit message: WIP
Parts:
- added C13: 0.1uF, Capacitor_SMD:C_0603_1608Metric_Pad1.08x0.95mm_HandSolder, B.Cu at (103.1, 103.5)
- added C14: 0.1uF, Capacitor_SMD:C_0603_1608Metric_Pad1.08x0.95mm_HandSolder, B.Cu at (88.5, 103.5)
- added C15: 0.1uF, Capacitor_SMD:C_0603_1608Metric_Pad1.08x0.95mm_HandSolder, B.Cu at (103.1, 97.8)
- added C16: 0.1uF, Capacitor_SMD:C_0603_1608Metric_Pad1.08x0.95mm_HandSolder, B.Cu at (88.5, 97.8)
- added J1: I/O EXPANSION, Connector_PCBEdge:BUS_PCIexpress_x4, F.Cu at (158.8, 106.7)
- added J2: PMOD1, Connector_PinSocket_2.54mm:PinSocket_2x06_P2.54mm_Horizontal, F.Cu at (116.9, 134.1)
- added J5: PMOD2, Connector_PinSocket_2.54mm:PinSocket_2x06_P2.54mm_Horizontal, F.Cu at (94.0, 134.1)
- added J6: PMOD3, Connector_PinSocket_2.54mm:PinSocket_2x06_P2.54mm_Horizontal, F.Cu at (129.6, 40.2)
- added J7: PMOD4, Connector_PinSocket_2.54mm:PinSocket_2x06_P2.54mm_Horizontal, F.Cu at (106.8, 40.2)
- C1, C12: footprint Capacitor_SMD:C_0805_2012Metric -> Capacitor_SMD:C_0603_1608Metric_Pad1.08x0.95mm_HandSolder
- C2, C3, C4, C5: footprint Capacitor_SMD:C_0805_2012Metric -> Capacitor_SMD:C_0603_1608Metric_Pad1.08x0.95mm_HandSolder; moved to B.Cu
- U2, U3: moved to B.Cu
- moved C10 141.5 mm to (69.6, 37.3), turned to -90 degrees
- moved C7 138.4 mm to (69.6, 31.9), turned to 90 degrees
- moved TP1 113.8 mm to (22.5, 61.5)
- moved TP4 113.8 mm to (22.3, 77.0)
- moved TP2 113.8 mm to (22.3, 68.8)
- moved TP3 113.8 mm to (28.7, 72.6)
- moved RN1 49.9 mm to (68.2, 70.4)
- moved U1 49.9 mm to (60.5, 65.2)
- moved PRIMER_20K_1 44.9 mm to (111.9, 87.5), turned to -90 degrees
- moved C1 43.3 mm to (64.3, 80.5), turned to 0 degrees
- moved R7 35.8 mm to (106.2, 160.0)
- moved D2 35.8 mm to (101.8, 160.1)
- moved C2 26.1 mm to (103.1, 81.7)
- moved J3 20.3 mm to (68.6, 46.4)
- moved C6 19.7 mm to (88.7, 158.2)
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Routing:
- added copper zone on B.Cu, net +3V3
- added copper zone on B.Cu, net +5V
Other:
- outline, holes or cut-outs redrawn
- board text added: "3v3"
- board text added: "6 8 0 9"
- board text added: "GND"
- board text removed: "6809"

Commit message: WIP
Parts:
- removed TP1: EXTAL, TestPoint:TestPoint_Loop_D1.80mm_Drill1.0mm_Beaded
- removed TP2: Q, TestPoint:TestPoint_Loop_D1.80mm_Drill1.0mm_Beaded
- removed TP3: E, TestPoint:TestPoint_Loop_D1.80mm_Drill1.0mm_Beaded
- removed TP4: R/~{W}, TestPoint:TestPoint_Loop_D1.80mm_Drill1.0mm_Beaded
- added C17: 10uF, Capacitor_SMD:C_0603_1608Metric_Pad1.08x0.95mm_HandSolder, F.Cu at (184.6, 66.0)
- added D3: WS2812B, LED_SMD:LED_WS2812B_PLCC4_5.0x5.0mm_P3.2mm, F.Cu at (86.3, 128.7)
- added D4: DSK24, Capacitor_SMD:C_0603_1608Metric_Pad1.08x0.95mm_HandSolder, F.Cu at (25.3, 86.9)
- added R10: 33, Resistor_SMD:R_0805_2012Metric, F.Cu at (185.4, 68.6)
- added R9: 33, Resistor_SMD:R_0805_2012Metric, F.Cu at (180.2, 66.3)
- added U5: HDSM-543B, Display:HDSM-541B_HDSM-543B, F.Cu at (67.3, 134.0)
- C6: footprint Capacitor_SMD:C_0805_2012Metric -> Capacitor_SMD:C_0603_1608Metric_Pad1.08x0.95mm_HandSolder
- J3: footprint Connector_PinHeader_2.54mm:PinHeader_2x06_P2.54mm_Vertical -> Connector_IDC:IDC-Header_2x06_P2.54mm_Vertical
- R8: value 50 -> 33
- moved SW2 52.1 mm to (48.2, 91.4)
- moved SW1 37.1 mm to (48.2, 104.1)
- moved SW3 5.89 mm to (86.4, 140.3)
- moved PRIMER_20K_1 4.96 mm to (107.0, 87.5)
- moved J3 3.17 mm to (71.1, 48.3)
Connections:
- net /BUF_A0 renamed /B_A0
- net /BUF_A1 renamed /B_A1
- net /BUF_A10 renamed /B_A10
- net /BUF_A11 renamed /B_A11
- net /BUF_A12 renamed /B_A12
- net /BUF_A13 renamed /B_A13
- net /BUF_A14 renamed /B_A14
- net /BUF_A15 renamed /B_A15
- net /BUF_A2 renamed /B_A2
- net /BUF_A3 renamed /B_A3
- net /BUF_A4 renamed /B_A4
- net /BUF_A5 renamed /B_A5
- net /BUF_A6 renamed /B_A6
- net /BUF_A7 renamed /B_A7
- net /BUF_A8 renamed /B_A8
- net /BUF_A9 renamed /B_A9
- net BUF_E renamed B_E
- net BUF_R/~{W} renamed B_R/~{W}
- net D_DIR renamed DIR
- net Net-(FB1-Pad2) renamed EXTAL
- J4 pad A4: +5V -> Net-(D4-A)
- J4 pad A9: +5V -> Net-(D4-A)
- J4 pad B4: +5V -> Net-(D4-A)
- J4 pad B9: +5V -> Net-(D4-A)
- R8 pad 1: Net-(R8-Pad1) -> Net-(FB1-Pad1)
- U1 pad 38: Net-(R8-Pad1) -> Net-(U1-EXTAL)
- U1 pad 7: +5V -> Net-(U1-VCC)
- U3 pad 44: unconnected-(U3-Pad44) -> Q
- U3 pad 5: unconnected-(U3-Pad5) -> B_Q
Other:
- copper layers 2 -> 4

Commit message: WIP
Parts:
- removed J2: PMOD1, Connector_PinSocket_2.54mm:PinSocket_2x06_P2.54mm_Horizontal
- removed J5: PMOD2, Connector_PinSocket_2.54mm:PinSocket_2x06_P2.54mm_Horizontal
- removed SW3: CONFIG, Button_Switch_SMD:SW_DIP_SPSTx04_Slide_KingTek_DSHP04TS_W7.62mm_P1.27mm
- removed U5: HDSM-543B, Display:HDSM-541B_HDSM-543B
- added D5: DSK24, Capacitor_SMD:C_0603_1608Metric_Pad1.08x0.95mm_HandSolder, F.Cu at (81.7, 40.6)
- added FB2: MPZ1608S101ATAH0, Capacitor_SMD:C_0603_1608Metric_Pad1.08x0.95mm_HandSolder, B.Cu at (53.7, 81.4)
- added U6: DLG-2416, footprints:DIP-18_W15.24mm_LongPads, F.Cu at (101.6, 141.6)
- C10: footprint Capacitor_SMD:C_0805_2012Metric -> Capacitor_SMD:C_0603_1608Metric_Pad1.08x0.95mm_HandSolder
- C13, C15, C2, C3: moved to F.Cu
- C17, C6: moved to B.Cu
- C8, C9: footprint Capacitor_SMD:C_0805_2012Metric -> Capacitor_SMD:C_0603_1608Metric_Pad1.08x0.95mm_HandSolder; moved to B.Cu
- R1, R10, R2, R3, R4, R5, R6, R8, R9: footprint Resistor_SMD:R_0805_2012Metric -> Resistor_SMD:R_0603_1608Metric_Pad0.98x0.95mm_HandSolder
- R7: footprint Resistor_SMD:R_0805_2012Metric -> Resistor_SMD:R_0603_1608Metric_Pad0.98x0.95mm_HandSolder; moved to B.Cu
- SW1: value FPGA_RST -> PTS636SK25SMTRLFS
- SW2: value MPU_RST -> PTS636SK25SMTRLFS
- moved C17 123.4 mm to (61.9, 80.0)
- moved C6 103.1 mm to (112.3, 57.8)
- moved R7 92.5 mm to (79.4, 71.5), turned to 180 degrees
- moved R8 82.7 mm to (147.8, 102.1)
- moved C9 78.6 mm to (48.2, 115.3), turned to -90 degrees
- moved C8 77.3 mm to (48.2, 128.0), turned to -90 degrees
- moved D4 60.8 mm to (54.0, 33.2), turned to -90 degrees
- moved D3 48.8 mm to (48.4, 97.9)
- moved R2 47.7 mm to (57.9, 165.9)
- moved D2 43.4 mm to (58.4, 162.3)
- moved R9 26.9 mm to (153.2, 66.0)
- moved R10 26.9 mm to (158.5, 68.3)
- moved H3 24.5 mm to (131.7, 33.3)
- moved J1 24.1 mm to (134.6, 106.7)
- moved H1 24.1 mm to (132.0, 141.0)
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Connections:
- C1 pad 1: +5V -> Net-(U1-VCC)
- C17 pad 1: +5V -> Net-(U1-VCC)
- H1 pad 1: unconnected-(H1-Pad1) -> GND
- H2 pad 1: unconnected-(H2-Pad1) -> GND
- H3 pad 1: unconnected-(H3-Pad1) -> GND
- H4 pad 1: unconnected-(H4-Pad1) -> GND
- J1 pad A1: (no net) -> +3V3
- J1 pad A10: (no net) -> ~{RESET}
- J1 pad A11: (no net) -> GND
- J1 pad A12: (no net) -> GND
- J1 pad A13: (no net) -> unconnected-(J1-Pin_a13-PadA13)
- J1 pad A14: (no net) -> unconnected-(J1-Pin_a14-PadA14)
- J1 pad A15: (no net) -> unconnected-(J1-Pin_a15-PadA15)
- J1 pad A16: (no net) -> unconnected-(J1-Pin_a16-PadA16)
- J1 pad A17: (no net) -> unconnected-(J1-Pin_a17-PadA17)
- J1 pad A18: (no net) -> unconnected-(J1-Pin_a18-PadA18)
- J1 pad A19: (no net) -> unconnected-(J1-Pin_a19-PadA19)
- J1 pad A2: (no net) -> +5V
- J1 pad A20: (no net) -> unconnected-(J1-Pin_a20-PadA20)
- J1 pad A21: (no net) -> unconnected-(J1-Pin_a21-PadA21)
- J1 pad A22: (no net) -> unconnected-(J1-Pin_a22-PadA22)
- J1 pad A23: (no net) -> unconnected-(J1-Pin_a23-PadA23)
- J1 pad A24: (no net) -> /B_D7
- J1 pad A25: (no net) -> /B_D6
- J1 pad A26: (no net) -> /B_D5
- J1 pad A27: (no net) -> /B_D4
- J1 pad A28: (no net) -> /B_D3
- J1 pad A29: (no net) -> /B_D2
- J1 pad A3: (no net) -> GND
- J1 pad A30: (no net) -> /B_D1
- J1 pad A31: (no net) -> /B_D0
- J1 pad A32: (no net) -> GND
- J1 pad A4: (no net) -> B_E
- J1 pad A5: (no net) -> B_Q
- J1 pad A6: (no net) -> unconnected-(J1-Pin_a6-PadA6)
- J1 pad A7: (no net) -> EXTAL
- J1 pad A8: (no net) -> unconnected-(J1-Pin_a8-PadA8)
- J1 pad A9: (no net) -> B_R/~{W}
- J1 pad B1: (no net) -> +3V3
- J1 pad B10: (no net) -> unconnected-(J1-Pin_b10-PadB10)
- J1 pad B11: (no net) -> GND
- J1 pad B12: (no net) -> GND
- J1 pad B13: (no net) -> /BUF_A15
- J1 pad B14: (no net) -> /BUF_A14
- J1 pad B15: (no net) -> /BUF_A13
- J1 pad B16: (no net) -> /BUF_A12
- J1 pad B17: (no net) -> /BUF_A11
- J1 pad B18: (no net) -> /BUF_A10
- J1 pad B19: (no net) -> /BUF_A9
- J1 pad B2: (no net) -> +5V
- J1 pad B20: (no net) -> /BUF_A8
- J1 pad B21: (no net) -> /BUF_A7
- J1 pad B22: (no net) -> /BUF_A6
- J1 pad B23: (no net) -> /BUF_A5
- J1 pad B24: (no net) -> /BUF_A4
- J1 pad B25: (no net) -> /BUF_A3
- J1 pad B26: (no net) -> /BUF_A2
- J1 pad B27: (no net) -> /BUF_A1
- J1 pad B28: (no net) -> /BUF_A0
- J1 pad B29: (no net) -> unconnected-(J1-Pin_b29-PadB29)
- J1 pad B3: (no net) -> GND
- J1 pad B30: (no net) -> unconnected-(J1-Pin_b30-PadB30)
- J1 pad B31: (no net) -> unconnected-(J1-Pin_b31-PadB31)
- J1 pad B32: (no net) -> GND
- J1 pad B4: (no net) -> GND
- J1 pad B5: (no net) -> GND
- J1 pad B6: (no net) -> ~{WRITE}
- J1 pad B7: (no net) -> ~{READ}
- J1 pad B8: (no net) -> unconnected-(J1-Pin_b8-PadB8)
- J1 pad B9: (no net) -> unconnected-(J1-Pin_b9-PadB9)
- J3 pad 11: /JTAG_TMS -> JTAG_TMS
- J3 pad 3: +5V -> Net-(D5-A)
- J3 pad 5: /JTAG_TCK -> JTAG_TCK
- J3 pad 6: /M11_IOR27B_FPGA_TXO -> FPGA_TX
- J3 pad 7: /JTAG_TDI -> JTAG_TDI
- J3 pad 8: /T13_IOR8B_FPGA_RXO -> FPGA_RX
- J3 pad 9: /JTAG_TDO -> JTAG_TDO
- PRIMER_20K_1 pad 1: /Tang Primer 20k Connector/T13_IOR8B_FPGA_RXO -> FPGA_RX
- PRIMER_20K_1 pad 11: /Tang Primer 20k Connector/M11_IOR27B_FPGA_TXO -> FPGA_TX
- PRIMER_20K_1 pad 143: /Tang Primer 20k Connector/JTAG_TMS -> JTAG_TMS
- PRIMER_20K_1 pad 147: /Tang Primer 20k Connector/JTAG_TDO -> JTAG_TDO
- PRIMER_20K_1 pad 149: /Tang Primer 20k Connector/JTAG_TCK -> JTAG_TCK
- PRIMER_20K_1 pad 153: /Tang Primer 20k Connector/JTAG_TDI -> JTAG_TDI
- U2 pad 11: /B_A6 -> /BUF_A6
- U2 pad 12: /B_A7 -> /BUF_A7
- U2 pad 13: /B_A8 -> /BUF_A8
- U2 pad 14: /B_A9 -> /BUF_A9
- U2 pad 16: /B_A10 -> /BUF_A10
- U2 pad 17: /B_A11 -> /BUF_A11
- U2 pad 19: /B_A12 -> /BUF_A12
- U2 pad 2: /B_A0 -> /BUF_A0
- U2 pad 20: /B_A13 -> /BUF_A13
- U2 pad 22: /B_A14 -> /BUF_A14
- U2 pad 23: /B_A15 -> /BUF_A15
- U2 pad 3: /B_A1 -> /BUF_A1
- U2 pad 5: /B_A2 -> /BUF_A2
- U2 pad 6: /B_A3 -> /BUF_A3
- U2 pad 8: /B_A4 -> /BUF_A4
- U2 pad 9: /B_A5 -> /BUF_A5
- U3 pad 13: /BUF_D0 -> /B_D0
- U3 pad 14: /BUF_D1 -> /B_D1
- U3 pad 16: /BUF_D2 -> /B_D2
- U3 pad 17: /BUF_D3 -> /B_D3
- U3 pad 19: /BUF_D4 -> /B_D4
- U3 pad 20: /BUF_D5 -> /B_D5
- U3 pad 22: /BUF_D6 -> /B_D6
- U3 pad 23: /BUF_D7 -> /B_D7
- U4 pad 8: /T13_IOR8B_FPGA_RXO -> FPGA_RX
- U4 pad 9: /M11_IOR27B_FPGA_TXO -> FPGA_TX
Routing:
- removed copper zone on B.Cu, net +3V3
- removed copper zone on B.Cu, net +5V
Other:
- board size 120 x 120 mm -> 95.9 x 120 mm

Commit message: wip
Parts:
- removed D2: 3V3, LED_SMD:LED_0805_2012Metric
- removed R2: 1k, Resistor_SMD:R_0603_1608Metric_Pad0.98x0.95mm_HandSolder
- added C18: 10uF, Capacitor_SMD:C_0603_1608Metric_Pad1.08x0.95mm_HandSolder, F.Cu at (163.3, 122.9)
- added C19: 0.1uF, Capacitor_SMD:C_0603_1608Metric_Pad1.08x0.95mm_HandSolder, F.Cu at (163.3, 125.4)
- added C20: 100nF, Capacitor_SMD:C_0603_1608Metric_Pad1.08x0.95mm_HandSolder, F.Cu at (163.3, 127.9)
- added C21: 10uF, Capacitor_SMD:C_0603_1608Metric_Pad1.08x0.95mm_HandSolder, B.Cu at (109.3, 142.7)
- added C22: 0.1uF, Capacitor_SMD:C_0603_1608Metric_Pad1.08x0.95mm_HandSolder, B.Cu at (106.6, 142.7)
- added C23: 10uF, Capacitor_SMD:C_0603_1608Metric_Pad1.08x0.95mm_HandSolder, B.Cu at (84.1, 142.8)
- added C24: 0.1uF, Capacitor_SMD:C_0603_1608Metric_Pad1.08x0.95mm_HandSolder, B.Cu at (81.3, 142.8)
- added J2: PS/2, footprints:DS1093-01, F.Cu at (130.6, 142.2)
- added J5: SERIAL, Connector_PinHeader_2.54mm:PinHeader_1x03_P2.54mm_Vertical, F.Cu at (130.8, 133.0)
- added J8: SERIAL, Connector_PinHeader_2.54mm:PinHeader_1x03_P2.54mm_Vertical, F.Cu at (89.5, 36.6)
- added R11: 10k, Resistor_SMD:R_0603_1608Metric_Pad0.98x0.95mm_HandSolder, F.Cu at (163.3, 130.4)
- added SW3: PWR, footprints:2UD1T1A1M2RES, F.Cu at (51.3, 45.7)
- added SW4: PTS636SK25SMTRLFS, Button_Switch_SMD:SW_SPST_CK_RS282G05A3, F.Cu at (163.3, 141.4)
- added U5: DLG-2416, footprints:DIP-18_W15.24mm_LongPads, F.Cu at (60.9, 146.7)
- added U7: WT32C3-01N, footprints:WT32C3, F.Cu at (145.9, 131.1)
- C14, C16, C4, C5: moved to F.Cu
- D5: value DSK24 -> WS2812B; footprint Capacitor_SMD:C_0603_1608Metric_Pad1.08x0.95mm_HandSolder -> LED_SMD:LED_WS2812B_PLCC4_5.0x5.0mm_P3.2mm
- J6: value PMOD3 -> PMOD4
- J7: value PMOD4 -> PMOD3
- moved D5 106.1 mm to (116.5, 140.8)
- moved D3 66.4 mm to (96.2, 51.9)
- moved R8 60.4 mm to (95.6, 71.8)
- moved U4 39.2 mm to (93.6, 42.8), turned to 90 degrees
- moved C12 39.2 mm to (89.5, 44.0)
- moved U6 16.2 mm to (86.3, 146.7)
- moved C16 15.5 mm to (95.0, 108.1), turned to 0 degrees
- moved H3 15.3 mm to (146.6, 37.0)
- moved H1 15.1 mm to (146.6, 144.8)
- moved J1 14.8 mm to (149.0, 110.5)
- moved C5 13.0 mm to (95.0, 81.7), turned to 0 degrees
- moved C4 12.7 mm to (94.7, 87.1), turned to 0 degrees
- moved J6 12.6 mm to (136.5, 44.1)
- moved J7 12.6 mm to (113.7, 44.1)
- moved C14 11.8 mm to (95.0, 101.3)
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- renumbered PRIMER_20K_1 to TANG_PRIMER_20K_1
Connections:
- net ~{DMA/BREQ} renamed ~{DMA}/~{BREQ}
- C8 pad 1: /T10_IOR35B_FPGA_~{RST} -> FPGA_~{RST}
- C9 pad 1: /LVDS_IOR53_N -> ~{RESET}
- D4 pad 1: +5V -> /5V_IN
- D5 pad 2: Net-(D5-A) -> unconnected-(D5-DOUT-Pad2)
- J1 pad A10: ~{RESET} -> unconnected-(J1-Pin_a10-PadA10)
- J1 pad A11: GND -> unconnected-(J1-Pin_a11-PadA11)
- J1 pad A13: unconnected-(J1-Pin_a13-PadA13) -> P11
- J1 pad A14: unconnected-(J1-Pin_a14-PadA14) -> P9
- J1 pad A15: unconnected-(J1-Pin_a15-PadA15) -> T9
- J1 pad A16: unconnected-(J1-Pin_a16-PadA16) -> P8
- J1 pad A17: unconnected-(J1-Pin_a17-PadA17) -> T8
- J1 pad A18: unconnected-(J1-Pin_a18-PadA18) -> R8
- J1 pad A19: unconnected-(J1-Pin_a19-PadA19) -> P6
- J1 pad A20: unconnected-(J1-Pin_a20-PadA20) -> T6
- J1 pad A21: unconnected-(J1-Pin_a21-PadA21) -> GND
- J1 pad A22: unconnected-(J1-Pin_a22-PadA22) -> /B_D7
- J1 pad A23: unconnected-(J1-Pin_a23-PadA23) -> /B_D6
- J1 pad A24: /B_D7 -> /B_D5
- J1 pad A25: /B_D6 -> /B_D4
- J1 pad A26: /B_D5 -> /B_D3
- J1 pad A27: /B_D4 -> /B_D2
- J1 pad A28: /B_D3 -> /B_D1
- J1 pad A29: /B_D2 -> /B_D0
- J1 pad A30: /B_D1 -> GND
- J1 pad A31: /B_D0 -> B_E
- J1 pad A32: GND -> B_Q
- J1 pad A4: B_E -> ~{RESET}
- J1 pad A5: B_Q -> unconnected-(J1-Pin_a5-PadA5)
- J1 pad A9: B_R/~{W} -> unconnected-(J1-Pin_a9-PadA9)
- J1 pad B10: unconnected-(J1-Pin_b10-PadB10) -> ~{READ}
- J1 pad B11: GND -> unconnected-(J1-Pin_b11-PadB11)
- J1 pad B13: /BUF_A15 -> unconnected-(J1-Pin_b13-PadB13)
- J1 pad B14: /BUF_A14 -> /B_A13
- J1 pad B15: /BUF_A13 -> /B_A14
- J1 pad B16: /BUF_A12 -> /B_A15
- J1 pad B17: /BUF_A11 -> /B_A12
- J1 pad B18: /BUF_A10 -> GND
- J1 pad B19: /BUF_A9 -> /B_A11
- J1 pad B20: /BUF_A8 -> /B_A10
- J1 pad B21: /BUF_A7 -> /B_A9
- J1 pad B22: /BUF_A6 -> /B_A8
- J1 pad B23: /BUF_A5 -> GND
- J1 pad B24: /BUF_A4 -> /B_A7
- J1 pad B25: /BUF_A3 -> /B_A6
- J1 pad B26: /BUF_A2 -> /B_A5
- J1 pad B27: /BUF_A1 -> /B_A4
- J1 pad B28: /BUF_A0 -> GND
- J1 pad B29: unconnected-(J1-Pin_b29-PadB29) -> /B_A3
- J1 pad B30: unconnected-(J1-Pin_b30-PadB30) -> /B_A2
- J1 pad B31: unconnected-(J1-Pin_b31-PadB31) -> /B_A1
- J1 pad B32: GND -> /B_A0
- J1 pad B6: ~{WRITE} -> unconnected-(J1-Pin_b6-PadB6)
- J1 pad B7: ~{READ} -> unconnected-(J1-Pin_b7-PadB7)
- J1 pad B8: unconnected-(J1-Pin_b8-PadB8) -> B_R/~{W}
- J1 pad B9: unconnected-(J1-Pin_b9-PadB9) -> ~{WRITE}
- J3 pad 3: Net-(D5-A) -> /5V_IN
- R3 pad 2: /T10_IOR35B_FPGA_~{RST} -> FPGA_~{RST}
- R6 pad 2: /LVDS_IOR53_N -> ~{RESET}
- SW1 pad 1: /T10_IOR35B_FPGA_~{RST} -> FPGA_~{RST}
- SW2 pad 1: /LVDS_IOR53_N -> ~{RESET}
- TANG_PRIMER_20K_1 pad 109: /Tang Primer 20k Connector/B14_IOL2A -> /B_A0
- TANG_PRIMER_20K_1 pad 113: /Tang Primer 20k Connector/A14_IOL8B -> /B_A1
- TANG_PRIMER_20K_1 pad 115: /Tang Primer 20k Connector/B13_IOL8A -> /B_A2
- TANG_PRIMER_20K_1 pad 119: /Tang Primer 20k Connector/C12_IOL7A -> /B_A3
- TANG_PRIMER_20K_1 pad 121: /Tang Primer 20k Connector/B12_IOL7B -> /B_A4
- TANG_PRIMER_20K_1 pad 123: /Tang Primer 20k Connector/A12_IOL13B -> /B_A5
- TANG_PRIMER_20K_1 pad 125: /Tang Primer 20k Connector/C11_IOL15B -> /B_A6
- TANG_PRIMER_20K_1 pad 129: /Tang Primer 20k Connector/B11_IOL13A -> /B_A7
- TANG_PRIMER_20K_1 pad 131: /Tang Primer 20k Connector/A11_IOL15A -> /B_A8
- TANG_PRIMER_20K_1 pad 135: /Tang Primer 20k Connector/C10_IOR39A -> /B_A9
- TANG_PRIMER_20K_1 pad 148: /Tang Primer 20k Connector/A9_IOL27A -> B_E
- TANG_PRIMER_20K_1 pad 15: /Tang Primer 20k Connector/T10_IOR35B_FPGA_~{RST} -> FPGA_~{RST}
- TANG_PRIMER_20K_1 pad 152: /Tang Primer 20k Connector/LVDS_IOT32_N -> ~{READ}
- TANG_PRIMER_20K_1 pad 154: /Tang Primer 20k Connector/LVDS_IOT32_P -> ~{WRITE}
- TANG_PRIMER_20K_1 pad 175: /Tang Primer 20k Connector/N6_IOR51A -> /B_A10
- TANG_PRIMER_20K_1 pad 177: /Tang Primer 20k Connector/N7_IOR47B -> /B_A11
- TANG_PRIMER_20K_1 pad 181: /Tang Primer 20k Connector/N9_IOR36B -> /B_A12
- TANG_PRIMER_20K_1 pad 183: /Tang Primer 20k Connector/R9_IOR35A -> /B_A15
- TANG_PRIMER_20K_1 pad 191: /Tang Primer 20k Connector/LVDS_IOR40_P -> /B_A14
- TANG_PRIMER_20K_1 pad 193: /Tang Primer 20k Connector/LVDS_IOR40_N -> /B_A13
- TANG_PRIMER_20K_1 pad 194: /Tang Primer 20k Connector/LVDS_IOR49_N -> DLG1_CS
- TANG_PRIMER_20K_1 pad 198: /Tang Primer 20k Connector/LVDS_IOR44_P -> DLG0_CS
- TANG_PRIMER_20K_1 pad 200: /Tang Primer 20k Connector/LVDS_IOR44_N -> DLG_~{BL}
- TANG_PRIMER_20K_1 pad 33: /Tang Primer 20k Connector/LVDS_IOR29_P -> B_Q
- TANG_PRIMER_20K_1 pad 39: /Tang Primer 20k Connector/LVDS_IOR42_N -> ~{HALT}
- TANG_PRIMER_20K_1 pad 45: /Tang Primer 20k Connector/LVDS_IOR38_P -> EXTAL
- TANG_PRIMER_20K_1 pad 50: /Tang Primer 20k Connector/LVDS_RX1_N -> T6
- TANG_PRIMER_20K_1 pad 52: /Tang Primer 20k Connector/LVDS_RX1_P -> P6
- TANG_PRIMER_20K_1 pad 56: /Tang Primer 20k Connector/LVDS_TX5_N -> R8
- TANG_PRIMER_20K_1 pad 58: /Tang Primer 20k Connector/LVDS_TX5_P -> T8
- TANG_PRIMER_20K_1 pad 62: /Tang Primer 20k Connector/LVDS_TX4_N -> P8
- TANG_PRIMER_20K_1 pad 64: /Tang Primer 20k Connector/LVDS_TX4_P -> T9
- TANG_PRIMER_20K_1 pad 67: /Tang Primer 20k Connector/LVDS_IOR20_P -> B_BS
- TANG_PRIMER_20K_1 pad 68: /Tang Primer 20k Connector/LVDS_TX3_P -> P9
- TANG_PRIMER_20K_1 pad 69: /Tang Primer 20k Connector/LVDS_IOR20_N -> B_BA
- TANG_PRIMER_20K_1 pad 70: /Tang Primer 20k Connector/LVDS_TX3_N -> P11
- TANG_PRIMER_20K_1 pad 74: /Tang Primer 20k Connector/LVDS_IOT38_N -> /B_D0
- TANG_PRIMER_20K_1 pad 76: /Tang Primer 20k Connector/LVDS_IOT38_P -> /B_D1
- TANG_PRIMER_20K_1 pad 77: /Tang Primer 20k Connector/LVDS_IOT8_P -> B_R/~{W}
- TANG_PRIMER_20K_1 pad 78: /Tang Primer 20k Connector/LVDS_IOT36_N -> /B_D2
- TANG_PRIMER_20K_1 pad 80: /Tang Primer 20k Connector/LVDS_IOT36_P -> /B_D3
- TANG_PRIMER_20K_1 pad 84: /Tang Primer 20k Connector/LVDS_IOT18_P -> /B_D4
- TANG_PRIMER_20K_1 pad 86: /Tang Primer 20k Connector/LVDS_IOT18_N -> /B_D5
- TANG_PRIMER_20K_1 pad 90: /Tang Primer 20k Connector/LVDS_IOT14_N -> /B_D6
- TANG_PRIMER_20K_1 pad 92: /Tang Primer 20k Connector/LVDS_IOT14_P -> /B_D7
- TANG_PRIMER_20K_1 pad 95: /Tang Primer 20k Connector/F14_IOT9A -> DIR
- U2 pad 11: /BUF_A6 -> /B_A6
- U2 pad 12: /BUF_A7 -> /B_A7
- U2 pad 13: /BUF_A8 -> /B_A8
- U2 pad 14: /BUF_A9 -> /B_A9
- U2 pad 16: /BUF_A10 -> /B_A10
- U2 pad 17: /BUF_A11 -> /B_A11
- U2 pad 19: /BUF_A12 -> /B_A12
- U2 pad 2: /BUF_A0 -> /B_A0
- U2 pad 20: /BUF_A13 -> /B_A15
- U2 pad 22: /BUF_A14 -> /B_A14
- U2 pad 23: /BUF_A15 -> /B_A13
- U2 pad 26: /A15 -> /A13
- U2 pad 29: /A13 -> /A15
- U2 pad 3: /BUF_A1 -> /B_A1
- U2 pad 5: /BUF_A2 -> /B_A2
- U2 pad 6: /BUF_A3 -> /B_A3
- U2 pad 8: /BUF_A4 -> /B_A4
- U2 pad 9: /BUF_A5 -> /B_A5
- U3 pad 12: unconnected-(U3-1B7-Pad12) -> B_R/~{W}
- U3 pad 2: B_R/~{W} -> unconnected-(U3-1B0-Pad2)
- U3 pad 3: B_E -> unconnected-(U3-1B1-Pad3)
- U3 pad 37: unconnected-(U3-1A7-Pad37) -> R/~{W}
- U3 pad 40: unconnected-(U3-1A5-Pad40) -> E
- U3 pad 41: unconnected-(U3-1A4-Pad41) -> Q
- U3 pad 43: unconnected-(U3-1A3-Pad43) -> BA
- U3 pad 44: Q -> BS
- U3 pad 46: E -> unconnected-(U3-1A1-Pad46)
- U3 pad 47: R/~{W} -> unconnected-(U3-1A0-Pad47)
- U3 pad 5: B_Q -> B_BS
- U3 pad 6: unconnected-(U3-1B3-Pad6) -> B_BA
- U3 pad 8: unconnected-(U3-1B4-Pad8) -> B_Q
- U3 pad 9: unconnected-(U3-1B5-Pad9) -> B_E
- U6 pad 1: DLG_CS -> DLG1_CS
- U6 pad 4: /BUF_A2 -> /B_A2
- U6 pad 6: /BUF_A3 -> /B_A3
- U6 pad 7: /BUF_A0 -> /B_A0
- U6 pad 8: /BUF_A1 -> /B_A1
Routing:
- net /B_A0: track 0.00 -> 168.7 mm, vias 0 -> 5
- net /B_A3: track 0.00 -> 166.9 mm, vias 0 -> 5
- net /B_A2: track 0.00 -> 163.9 mm, vias 0 -> 6
- net /B_A1: track 0.00 -> 160.8 mm, vias 0 -> 6
- net /B_D0: track 0.00 -> 155.4 mm, vias 0 -> 5
- net /B_D1: track 0.00 -> 151.6 mm, vias 0 -> 5
- net /B_D2: track 0.00 -> 148.9 mm, vias 0 -> 5
- net /B_D3: track 0.00 -> 146.2 mm, vias 0 -> 5
- net /B_D4: track 0.00 -> 141.2 mm, vias 0 -> 4
- net /B_D5: track 0.00 -> 140.2 mm, vias 0 -> 4
- net /B_D6: track 0.00 -> 138.5 mm, vias 0 -> 4
- net JTAG_TCK: track 0.00 -> 90.4 mm, vias 0 -> 2
- net JTAG_TDI: track 0.00 -> 89.7 mm, vias 0 -> 2
- net JTAG_TMS: track 0.00 -> 83.6 mm, vias 0 -> 2
- net JTAG_TDO: track 0.00 -> 82.4 mm, vias 0 -> 2
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- added copper zone on In2.Cu, net +3V3
- added copper zone on In2.Cu, net +5V
- added copper zone on In1.Cu, net GND
Other:
- board size 95.9 x 120 mm -> 105.9 x 120 mm
- board text added: "Anachron"
- board text added: "RX"
- board text added: "TX"
- board text added: "⍺"
- board text removed: "6 8 0 9"

Commit message: WIP
Parts:
- D1: footprint LED_SMD:LED_0805_2012Metric -> LED_SMD:LED_0603_1608Metric_Pad1.05x0.95mm_HandSolder
- moved R1 111.6 mm to (56.5, 51.8), turned to -90 degrees
- moved D1 105.4 mm to (52.6, 55.0), turned to 180 degrees
- moved U7 29.2 mm to (174.9, 134.9), turned to 90 degrees
- moved D4 4.09 mm to (57.9, 41.1), turned to 0 degrees
- moved C12 2.79 mm to (90.4, 41.4)
- moved R8 1.17 mm to (94.9, 70.9)
- moved R4 0.86 mm to (64.4, 43.4)
- moved R5 0.71 mm to (67.9, 43.4)
Connections:
- C9 pad 1: ~{RESET} -> MPU_~{RST}
- J1 pad A7: EXTAL -> unconnected-(J1-Pin_a7-PadA7)
- J1 pad B11: unconnected-(J1-Pin_b11-PadB11) -> GND
- J1 pad B4: GND -> unconnected-(J1-Pin_b4-PadB4)
- J1 pad B5: GND -> unconnected-(J1-Pin_b5-PadB5)
- J1 pad B6: unconnected-(J1-Pin_b6-PadB6) -> E_EXTAL
- R6 pad 2: ~{RESET} -> MPU_~{RST}
- RN1 pad 10: (no net) -> unconnected-(RN1-NC-Pad10)
- SW2 pad 1: ~{RESET} -> MPU_~{RST}
- TANG_PRIMER_20K_1 pad 148: B_E -> /Tang Primer 20k Connector/A9_IOL27A
- TANG_PRIMER_20K_1 pad 158: /Tang Primer 20k Connector/E9_IOL38B_1V5 -> E_EXTAL
- TANG_PRIMER_20K_1 pad 27: /Tang Primer 20k Connector/LVDS_IOR53_N -> MPU_~{RST}
- TANG_PRIMER_20K_1 pad 33: B_Q -> /Tang Primer 20k Connector/LVDS_IOR29_P
- TANG_PRIMER_20K_1 pad 44: /Tang Primer 20k Connector/LVDS_RX2_P -> B_Q
- TANG_PRIMER_20K_1 pad 46: /Tang Primer 20k Connector/LVDS_RX2_N -> B_E
- TANG_PRIMER_20K_1 pad 53: /Tang Primer 20k Connector/LVDS_IOR24_P -> ~{RESET}
- U5 pad 5: (no net) -> unconnected-(U5-NC-Pad5)
- U6 pad 5: (no net) -> unconnected-(U6-NC-Pad5)
Routing:
- net ~{RESET}: track 40.1 -> 235.8 mm, vias 0 -> 5
- net FPGA_~{RST}: track 0.00 -> 130.7 mm, vias 0 -> 3
- net +5V: track 11.4 -> 136.3 mm, vias 4 -> 8
- net MPU_~{RST}: track 0.00 -> 119.0 mm, vias 0 -> 3
- net +3V3: track 31.0 -> 91.6 mm, vias 11 -> 15
- net B_R/~{W}: track 6.41 -> 65.1 mm, vias 1 -> 3
- net /5V_IN: track 0.00 -> 40.6 mm
- net D-: track 0.00 -> 38.8 mm
- net D+: track 0.00 -> 37.2 mm, vias 0 -> 2
- net E_EXTAL: track 0.00 -> 36.7 mm
- net Net-(D4-A): track 0.00 -> 16.1 mm, vias 0 -> 2
- net GND: track 46.1 -> 50.5 mm, vias 33 -> 36
- net Net-(J4-CC1): track 0.00 -> 3.79 mm
- net Net-(J4-CC2): track 0.00 -> 3.56 mm
- net B_E: track 61.3 -> 64.2 mm
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