File: Tang20k_con.kicad_sch (KiCad schematic)
At the start: 1 part

Commit message: WIP
Connections:
- net M11_IOR27B_FPGA_TXO renamed FPGA_TX
- net T13_IOR8B_FPGA_RXO renamed FPGA_RX
Other:
- moved on the sheet: PRIMER_20K_1A

Commit message: wip
Parts:
- renumbered PRIMER_20K_1 to TANG_PRIMER_20K_1
Connections:
- net A9_IOL27A is gone; now on net B_E: TANG_PRIMER_20K_1.148
- net F14_IOT9A is gone; now on net DIR: TANG_PRIMER_20K_1.95
- net LVDS_IOR29_P is gone; now on net B_Q: TANG_PRIMER_20K_1.33
- net LVDS_IOR38_P is gone; now on net EXTAL: TANG_PRIMER_20K_1.45
- net LVDS_IOT8_P is gone; now on net B_R/~{W}: TANG_PRIMER_20K_1.77
- net C10_IOR39A renamed B_A9
- net C11_IOL15B renamed B_A6
- net C12_IOL7A renamed B_A3
- net LVDS_IOR20_N renamed B_BA
- net LVDS_IOR20_P renamed B_BS
- net LVDS_IOR40_N renamed B_A13
- net LVDS_IOR40_P renamed B_A14
- net LVDS_IOR42_N renamed ~{HALT}
- net LVDS_IOR44_N renamed DLG_~{BL}
- net LVDS_IOR44_P renamed DLG0_CS
- net LVDS_IOR49_N renamed DLG1_CS
- net LVDS_IOT14_N renamed B_D6
- net LVDS_IOT14_P renamed B_D7
- net LVDS_IOT18_N renamed B_D5
- net LVDS_IOT18_P renamed B_D4
- net LVDS_IOT32_N renamed ~{READ}
- net LVDS_IOT32_P renamed ~{WRITE}
- net LVDS_IOT36_N renamed B_D2
- net LVDS_IOT36_P renamed B_D3
- net LVDS_IOT38_N renamed B_D0
- net LVDS_IOT38_P renamed B_D1
- net LVDS_RX1_N renamed T6
- net LVDS_RX1_P renamed P6
- net LVDS_TX3_N renamed P11
- net LVDS_TX3_P renamed P9
- net LVDS_TX4_N renamed P8
- net LVDS_TX4_P renamed T9
- net LVDS_TX5_N renamed R8
- net LVDS_TX5_P renamed T8
- net N6_IOR51A renamed B_A10
- net N7_IOR47B renamed B_A11
- net N9_IOR36B renamed B_A12
- net R9_IOR35A renamed B_A15
- net T10_IOR35B_FPGA_~{RST} renamed FPGA_~{RST}
- no-connect marks 40 -> 46
Other:
- note added: "4,5,6 = 1.5v"
- moved on the sheet: TANG_PRIMER_20K_1A, TANG_PRIMER_20K_1B

Commit message: WIP
Connections:
- net LVDS_IOR24_P is gone; now on net ~{RESET}: TANG_PRIMER_20K_1.53
- net LVDS_RX2_N is gone; now on net B_E: TANG_PRIMER_20K_1.46
- net LVDS_RX2_P is gone; now on net B_Q: TANG_PRIMER_20K_1.44
- net B_E: no longer TANG_PRIMER_20K_1.148
- net B_Q: no longer TANG_PRIMER_20K_1.33
- net E9_IOL38B_1V5 renamed E_EXTAL
- net LVDS_IOR53_N renamed MPU_~{RST}
- new net A9_IOL27A: TANG_PRIMER_20K_1.148
- new net LVDS_IOR29_P: TANG_PRIMER_20K_1.33
Changed lines of the file:
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@@
+    (stroke (width 0) (type default))
+  )
+  (wire (pts (xy 231.775 98.425) (xy 259.08 98.425))
     (stroke (width 0) (type default))
   )
@@
     (stroke (width 0) (type default))
   )
-  (wire (pts (xy 240.919 95.885) (xy 231.775 95.885))
+  (wire (pts (xy 259.08 95.885) (xy 231.775 95.885))
     (stroke (width 0) (type default))
   )
@@
     (stroke (width 0) (type default))
   )
-  (wire (pts (xy 112.395 132.08) (xy 107.315 132.08))
+  (wire (pts (xy 107.315 132.08) (xy 138.43 132.08))
     (stroke (width 0) (type default))
   )
@@
     (stroke (width 0) (type default))
   )
+  (wire (pts (xy 176.53 108.585) (xy 211.455 108.585))
+    (stroke (width 0) (type default))
+  )
   (wire (pts (xy 231.775 111.125) (xy 259.08 111.125))
     (stroke (width 0) (type default))
@@
     (stroke (width 0) (type default))
   )
-  (wire (pts (xy 114.935 167.64) (xy 107.315 167.64))
+  (wire (pts (xy 138.43 167.64) (xy 107.315 167.64))
     (stroke (width 0) (type default))
   )
@@
     )
   )
-  (global_label "~{RESET}" (shape output) (at 140.97 231.775 180) (fields_autoplaced)
+  (global_label "~{RESET}" (shape output) (at 176.53 108.585 180) (fields_autoplaced)
     (effects (font (size 1.27 1.27)) (justify right))
-    (property "Intersheetrefs" "${INTERSHEET_REFS}" (at 132.3191 231.775 0)
+    (property "Intersheetrefs" "${INTERSHEET_REFS}" (at 167.8791 108.585 0)
       (effects (font (size 1.27 1.27)) (justify right) hide)
     )
@@
     )
   )
+  (global_label "MPU_~{RST}" (shape input) (at 176.53 75.565 180) (fields_autoplaced)
+    (effects (font (size 1.27 1.27)) (justify right))
+    (property "Intersheetrefs" "${INTERSHEET_REFS}" (at 165.1576 75.565 0)
+      (effects (font (size 1.27 1.27)) (justify right) hide)
+    )
+  )
   (global_label "FPGA_TX" (shape output) (at 176.53 55.245 180) (fields_autoplaced)
     (effects (font (size 1.27 1.27)) (justify right))
@@
     )
   )
+  (global_label "E_EXTAL" (shape input) (at 138.43 132.08 0) (fields_autoplaced)
+    (effects (font (size 1.27 1.27)) (justify left))
+    (property "Intersheetrefs" "${INTERSHEET_REFS}" (at 148.8952 132.08 0)
+      (effects (font (size 1.27 1.27)) (justify left) hide)
+    )
+  )
   (global_label "~{DMA}{slash}~{BREQ}" (shape input) (at 142.875 225.425 180) (fields_autoplaced)
     (effects (font (size 1.27 1.27)) (justify right))
@@
     )
   )
-  (global_label "B_Q" (shape input) (at 176.53 83.185 180) (fields_autoplaced)
-    (effects (font (size 1.27 1.27)) (justify right))
-    (property "Intersheetrefs" "${INTERSHEET_REFS}" (at 170.0561 83.185 0)
-      (effects (font (size 1.27 1.27)) (justify right) hide)
+  (global_label "B_Q" (shape input) (at 259.08 95.885 0) (fields_autoplaced)
+    (effects (font (size 1.27 1.27)) (justify left))
+    (property "Intersheetrefs" "${INTERSHEET_REFS}" (at 265.5539 95.885 0)
+      (effects (font (size 1.27 1.27)) (justify left) hide)
     )
   )
@@
     )
   )
-  (global_label "B_E" (shape input) (at 138.43 119.38 0) (fields_autoplaced)
+  (global_label "B_E" (shape input) (at 259.08 98.425 0) (fields_autoplaced)
     (effects (font (size 1.27 1.27)) (justify left))
-    (property "Intersheetrefs" "${INTERSHEET_REFS}" (at 144.2298 119.3006 0)
+    (property "Intersheetrefs" "${INTERSHEET_REFS}" (at 264.8798 98.3456 0)
       (effects (font (size 1.27 1.27)) (justify left) hide)
     )

Commit message: WIP
Connections:
- net LVDS_IOR17_N is gone; now on net E_O: TANG_PRIMER_20K_1.59
- net LVDS_IOR17_P is gone; now on net Q_O: TANG_PRIMER_20K_1.57
Changed lines of the file:
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@@
+    (stroke (width 0) (type default))
+  )
+  (wire (pts (xy 176.53 113.665) (xy 211.455 113.665))
     (stroke (width 0) (type default))
   )
@@
   )
   (wire (pts (xy 138.43 124.46) (xy 107.315 124.46))
+    (stroke (width 0) (type default))
+  )
+  (wire (pts (xy 176.53 116.205) (xy 211.455 116.205))
     (stroke (width 0) (type default))
   )
@@
     )
   )
-  (global_label "Q_O" (shape output) (at 129.54 230.505 180) (fields_autoplaced)
-    (effects (font (size 1.27 1.27)) (justify right))
-    (property "Intersheetrefs" "${INTERSHEET_REFS}" (at 123.0056 230.505 0)
+  (global_label "Q_O" (shape output) (at 176.53 113.665 180) (fields_autoplaced)
+    (effects (font (size 1.27 1.27)) (justify right))
+    (property "Intersheetrefs" "${INTERSHEET_REFS}" (at 169.9956 113.665 0)
       (effects (font (size 1.27 1.27)) (justify right) hide)
     )
@@
     )
   )
-  (global_label "E_O" (shape output) (at 129.54 233.045 180) (fields_autoplaced)
-    (effects (font (size 1.27 1.27)) (justify right))
-    (property "Intersheetrefs" "${INTERSHEET_REFS}" (at 123.1871 233.045 0)
-      (effects (font (size 1.27 1.27)) (justify right) hide)
-    )
+  (global_label "E_O" (shape output) (at 176.53 116.205 180) (fields_autoplaced)
+    (effects (font (size 1.27 1.27)) (justify right))
+    (property "Intersheetrefs" "${INTERSHEET_REFS}" (at 170.1771 116.205 0)
+      (effects (font (size 1.27 1.27)) (justify right) hide)
+    )

Commit message: WIP
Connections:
- net A15_IOL2B is gone; now on net ~{DMA}/~{BREQ}: TANG_PRIMER_20K_1.107
- net F16_IOT9B is gone; now on net ~{NMI}: TANG_PRIMER_20K_1.97
- net LVDS_IOR24_N is gone; now on net P11: TANG_PRIMER_20K_1.51
- net LVDS_IOR29_N is gone; now on net R8: TANG_PRIMER_20K_1.35
- net LVDS_IOR38_N is gone; now on net P9: TANG_PRIMER_20K_1.47
- net LVDS_IOR42_P is gone; now on net P8: TANG_PRIMER_20K_1.41
- net LVDS_IOR53_P is gone; now on net P6: TANG_PRIMER_20K_1.29
- net LVDS_IOT44_N is gone; now on net ~{IRQ}: TANG_PRIMER_20K_1.101
- net LVDS_IOT44_P is gone; now on net ~{FIRQ}: TANG_PRIMER_20K_1.103
- net P11: no longer TANG_PRIMER_20K_1.70
- net P6: no longer TANG_PRIMER_20K_1.52
- net P8: no longer TANG_PRIMER_20K_1.62
- net P9: no longer TANG_PRIMER_20K_1.68
- net R8: no longer TANG_PRIMER_20K_1.56
- net E10_IOL17B renamed KBD_DATA
- net LVDS_IOR11_N renamed P13
- net LVDS_IOR11_P renamed R12
- net LVDS_IOR29_P renamed T7
- net LVDS_IOR49_P renamed KBD_CLK
- net LVDS_IOT40_N renamed M15
- net LVDS_IOT40_P renamed M14
- net LVDS_RX3_N renamed N14
- net LVDS_RX3_P renamed N16
- net LVDS_RX4_N renamed P16
- net LVDS_RX4_P renamed N15
- net LVDS_RX5_N renamed R16
- net LVDS_RX5_P renamed P15
- net T6 renamed K15
- net T8 renamed J15
- net T9 renamed H14
- new net G16: TANG_PRIMER_20K_1.68
- new net H15: TANG_PRIMER_20K_1.70
- new net H16: TANG_PRIMER_20K_1.62
- new net K14: TANG_PRIMER_20K_1.52
- new net K16: TANG_PRIMER_20K_1.56
Other:
- note added: "3/IOR42B/P8"
- note removed: "3/IOR42B/M6"
