File: io.kicad_sch (KiCad schematic)
At the start: 13 parts, among them J2 PS/2, J5 SERIAL, J6 PMOD3, J7 PMOD4, SW4 PTS636SK25SMTRLFS, SW5 SW_DIP_x04, U7 WT32C3-01N

Commit message: WIP
Parts:
- removed SW5: SW_DIP_x04, symbol Switch:SW_DIP_x04
Other:
- moved on the sheet: C18, C19, C20, J5, R11, SW4, U7

Commit message: WIP
Parts:
- removed U7: WT32C3-01N, footprints:WT32C3, symbol custom6309:WT32C3-01N
- added R11 (x2): 2k, Resistor_SMD:R_0603_1608Metric_Pad0.98x0.95mm_HandSolder, symbol Device:R_Small_US
- added TP1: E, TestPoint:TestPoint_THTPad_D1.0mm_Drill0.5mm, symbol Connector:TestPoint_Small
- added TP2: Q, TestPoint:TestPoint_THTPad_D1.0mm_Drill0.5mm, symbol Connector:TestPoint_Small
Connections:
- net +3V3: now also R11.1, R11.1
- net KBD_CLK: now also R11.2
- net KBD_DATA: now also R11.2
- net N15: now reaches J7.10 (Pin_10)
- net P15: now reaches J7.11 (Pin_11)
- net R16: now reaches J7.12 (Pin_12)
- net M15: now reaches J7.5 (Pin_5)
- net M14: now reaches J7.6 (Pin_6)
- net N16: now reaches J7.7 (Pin_7)
- net N14: now reaches J7.8 (Pin_8)
- net P16: now reaches J7.9 (Pin_9)
- net P8: now reaches J6.10 (Pin_10)
- net P6: now reaches J6.11 (Pin_11)
- net T7: now reaches J6.12 (Pin_12)
- net R12: now reaches J6.5 (Pin_5)
- net P13: now reaches J6.6 (Pin_6)
- net P9: now reaches J6.7 (Pin_7)
- net P11: now reaches J6.8 (Pin_8)
- net R8: now reaches J6.9 (Pin_9)
- new net B_E: TP1.1
- new net B_Q: TP2.1
